File: pcb/BurnedHead.kicad_pcb (KiCad board)
At the start: 4 copper layers, 121.9 x 44.4 mm, 92 parts, among them J1 USB_B_Micro, J2 Conn_ARM_JTAG_SWD_10, J3 DM3AT-SF-PEJMS, J4 FPC_1x5_TopContact_P=0.5mm, J5 FPC_1x5_TopContact_P=0.5mm, Q2 IRLML6401TRPBF, SW1 SW_SPDT, SW2 SW_Push, SW3 SW_Push, SW4 DualShock-DPad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

Commit message: Move to kicad 5.99 nightly
Other:
- net class Default removed
- net class IC_POWER removed
- net class LCD removed
- net class SDRAM_DQ removed
- net class VSUPPLY removed
